Commit message: Multiple robots working without cameras

File: robotiq_description/urdf/robotiq_2f_85_macro.urdf.xacro (robot description, xacro)
@@ -163,7 +163,9 @@
                 </geometry>
             </visual>
-            <collision>
-                <geometry>
-                    <mesh filename="package://robotiq_description/meshes/collision/2f_85/left_finger_tip.stl" />
+            <!-- Box primitive matches collision STL AABB; tighter Bullet contact than tri-mesh. -->
+            <collision>
+                <origin xyz="-0.00965 -0.0008 0.02252" rpy="0 0 0" />
+                <geometry>
+                    <box size="0.0312 0.027 0.057" />
                 </geometry>
                 <surface>
@@ -199,6 +201,7 @@
             </visual>
             <collision>
-                <geometry>
-                    <mesh filename="package://robotiq_description/meshes/collision/2f_85/right_finger_tip.stl" />
+                <origin xyz="0.00965 0.00005 0.02252" rpy="0 0 0" />
+                <geometry>
+                    <box size="0.0312 0.027 0.057" />
                 </geometry>
                 <surface>
